File: Li-Po Charger.kicad_sch (KiCad schematic)
At the start: 31 parts, among them J1 USB_C_Receptacle_PowerOnly_6P, J2 JST_2mm_LiPo, J3 I^{2}C 1, J4 I^{2}C 2, J5 I^{2}C 3, J6 Inputs, J7 Outputs, Q1 IRLML6401, U1 MAX17048, U2 ME6211C33M5, U3 TP4056-42-ESOP8

Commit message: Revise the board following a design review
With R1 at 10K the load ran through Q1's body diode for about 35 ms
after USB was unplugged; 1.5K shortens that to about 5 ms. A USB host
expects about 10 uF at plug-in, and C3 was the part of it that could
shrink. Plug-in ringing on VBUS reaches the LDO through D1, and the
LDO's 6.5 V limit is the lowest on that rail.

PWR_OFF and CHRG_OFF are pulled up, so the 3.3 V rail and charging are
on until a pin is driven low.

The LDO cannot feed an amplifier or a motor, which take V_SYS or the
battery from J8. A track running down to J8 on the back cuts the ground
pour that joins the USB side to the battery side, so the battery and
V_SYS reach it on the front and 5 V crosses on the back.

J2's mounting pad was inside the edge clearance. The board file is in
KiCad 10's format, which KiCad 9 cannot open.
Parts:
- added D2: SD05, Diode_SMD:D_SOD-323, symbol Diode:ESD5Zxx
- added J8: Power, Connector_PinHeader_2.54mm:PinHeader_1x04_P2.54mm_Vertical, symbol Connector_Generic:Conn_01x04
- C3: value 10uF -> 1uF
- J6: value Inputs -> Control; footprint Connector_PinHeader_2.54mm:PinHeader_1x04_P2.54mm_Vertical -> Connector_PinHeader_2.54mm:PinHeader_1x03_P2.54mm_Vertical; symbol Connector_Generic:Conn_01x04 -> Connector_Generic:Conn_01x03
- J7: value Outputs -> Status
- R1: value 10K -> 1.5K
- RV1: LCSC Part C719176 -> (none); LCSC Part # (none) -> C719176
Connections:
- net +5V: now also D2.1 (K), J8.1 (Pin_1); no longer J6.3 (Pin_3)
- net +BATT: now also J8.2 (Pin_2)
- net GND: now also J6.3 (Pin_3), D2.2 (A), J8.4 (Pin_4); no longer J6.4 (Pin_4)
- net V_{SYS}: now also J8.3 (Pin_3)
- net CHARGE_EN renamed ~{CHRG_OFF}
- net POWER_EN renamed ~{PWR_OFF}
